File: dilemma_assembled/dilemma.kicad_pcb (KiCad board)
At the start: 2 copper layers, 134.1 x 110.3 mm, 124 parts, among them J1 USB_C_Receptacle_USB2.0, J102 Serial, J103 Serial, J105 Conn_01x04_Female, J107 Conn_01x08_Female, J108 Conn_01x01_Female, J109 Conn_01x01_Female, J113 Cirque, J5 Conn_01x02, SW1 SW_Push, SW101 SW_Push, SW102 SW_Push, SW103 SW_Push, SW104 SW_Push, SW105 SW_Push, SW106 SW_Push, SW107 SW_Push, SW108 SW_Push, SW109 SW_Push, SW110 SW_SPST, SW111 SW_SPST, SW112 SW_Push, SW113 SW_Push, SW114 SW_Push, SW115 SW_Push, SW116 SW_Push, SW117 SW_Push, SW118 SW_Push, SW119 locked, SW2 SW_Push, U1 RP2040, U2 GD25Q80CEIGR, U3 XC6210B332MR-G, Y1 Crystal_GND24

Commit message: add 6th column
Parts:
- removed the REF** at (100.4, 59.2)
- added D118: D, local-libraries:D_1206_handsolder_reversible, F.Cu at (43.5, 54.6)
- added D119: D, local-libraries:D_1206_handsolder_reversible, F.Cu at (43.6, 73.7)
- added D120: D, local-libraries:D_1206_handsolder_reversible, F.Cu at (44.1, 92.2)
- added SW120: SW_Push, local-libraries:SW_MX_choc, F.Cu at (34.4, 53.7)
- added SW121: SW_Push, local-libraries:SW_MX_choc, F.Cu at (34.4, 72.7)
- added SW122: SW_Push, local-libraries:SW_MX_choc, F.Cu at (34.4, 91.7)
Connections:
- U1 pad 15: /D12 -> col6_l
Routing:
- net col6_l: track 0.00 -> 177.8 mm, vias 0 -> 2
- net row2_l: track 197.8 -> 241.2 mm
- net row3_l: track 213.2 -> 254.4 mm
- net row4_l: track 230.2 -> 266.9 mm
- net Net-(D120-Pad2): track 0.00 -> 25.5 mm
- net Net-(D119-Pad2): track 0.00 -> 25.5 mm
- net Net-(D118-Pad2): track 0.00 -> 25.5 mm
Other:
- board size 134.1 x 110.3 mm -> 153.1 x 110.3 mm
- board text added: "3x6_a1.1a"
- board text removed: "a1.1c"
