File: dilemma_assembled/dilemma.kicad_pcb (KiCad board)
At the start: 2 copper layers, 153.1 x 110.3 mm, 129 parts, among them J1 USB_C_Receptacle_USB2.0, J102 Serial, J103 Serial, J105 Conn_01x04_Female, J107 Conn_01x08_Female, J108 Conn_01x01_Female, J109 Conn_01x01_Female, J113 Cirque, J5 Conn_01x02, SW1 SW_Push, SW101 SW_Push, SW102 SW_Push, SW103 SW_Push, SW104 SW_Push, SW105 SW_Push, SW106 SW_Push, SW107 SW_Push, SW108 SW_Push, SW109 SW_Push, SW110 SW_SPST, SW111 SW_SPST, SW112 SW_Push, SW113 SW_Push, SW114 SW_Push, SW115 SW_Push, SW116 SW_Push, SW117 SW_Push, SW118 SW_Push, SW119 locked, SW120 SW_Push, SW121 SW_Push, SW122 SW_Push, SW2 SW_Push, U1 RP2040, U2 GD25Q80CEIGR, U3 XC6210B332MR-G, Y1 Crystal_GND24

Commit message: annotate schematic
Changed lines of the file:
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@@
     (pad "1" thru_hole circle (at -2.25 0 90) (size 0.5 0.5) (drill 0.3) (layers *.Cu *.Mask)
       (net 26 "col6_l") (pinfunction "K") (pintype "passive"))
-    (pad "1" smd roundrect (at -1.4875 0 90) (size 1.425 1.75) (layers "F.Cu" "F.Paste" "F.Mask") (roundrect_rratio 0.175439)
+    (pad "1" smd roundrect (at -1.4875 0 90) (size 1.425 1.75) (layers "F.Cu" "F.Paste" "F.Mask") (roundrect_rratio 0.1754392982)
       (net 26 "col6_l") (pinfunction "K") (pintype "passive"))
-    (pad "2" smd roundrect (at 1.4875 0 90) (size 1.425 1.75) (layers "F.Cu" "F.Paste" "F.Mask") (roundrect_rratio 0.175439)
+    (pad "2" smd roundrect (at 1.4875 0 90) (size 1.425 1.75) (layers "F.Cu" "F.Paste" "F.Mask") (roundrect_rratio 0.1754392982)
       (net 92 "Net-(D119-Pad2)") (pinfunction "A") (pintype "passive"))
     (pad "2" thru_hole circle (at 2.2 0 90) (size 0.5 0.5) (drill 0.3) (layers *.Cu *.Mask)
@@
     (pad "1" thru_hole circle (at -2.25 0 90) (size 0.5 0.5) (drill 0.3) (layers *.Cu *.Mask)
       (net 26 "col6_l") (pinfunction "K") (pintype "passive"))
-    (pad "1" smd roundrect (at -1.4875 0 90) (size 1.425 1.75) (layers "F.Cu" "F.Paste" "F.Mask") (roundrect_rratio 0.175439)
+    (pad "1" smd roundrect (at -1.4875 0 90) (size 1.425 1.75) (layers "F.Cu" "F.Paste" "F.Mask") (roundrect_rratio 0.1754392982)
       (net 26 "col6_l") (pinfunction "K") (pintype "passive"))
     (pad "2" thru_hole circle (at 2.2 0 90) (size 0.5 0.5) (drill 0.3) (layers *.Cu *.Mask)
       (net 93 "Net-(D120-Pad2)") (pinfunction "A") (pintype "passive"))
-    (pad "2" smd roundrect (at 1.4875 0 90) (size 1.425 1.75) (layers "F.Cu" "F.Paste" "F.Mask") (roundrect_rratio 0.175439)
+    (pad "2" smd roundrect (at 1.4875 0 90) (size 1.425 1.75) (layers "F.Cu" "F.Paste" "F.Mask") (roundrect_rratio 0.1754392982)
       (net 93 "Net-(D120-Pad2)") (pinfunction "A") (pintype "passive"))
   )
@@
     (pad "1" thru_hole circle (at -2.25 0 90) (size 0.5 0.5) (drill 0.3) (layers *.Cu *.Mask)
       (net 26 "col6_l") (pinfunction "K") (pintype "passive"))
-    (pad "1" smd roundrect (at -1.4875 0 90) (size 1.425 1.75) (layers "F.Cu" "F.Paste" "F.Mask") (roundrect_rratio 0.175439)
+    (pad "1" smd roundrect (at -1.4875 0 90) (size 1.425 1.75) (layers "F.Cu" "F.Paste" "F.Mask") (roundrect_rratio 0.1754392982)
       (net 26 "col6_l") (pinfunction "K") (pintype "passive"))
     (pad "2" thru_hole circle (at 2.2 0 90) (size 0.5 0.5) (drill 0.3) (layers *.Cu *.Mask)
       (net 91 "Net-(D118-Pad2)") (pinfunction "A") (pintype "passive"))
-    (pad "2" smd roundrect (at 1.4875 0 90) (size 1.425 1.75) (layers "F.Cu" "F.Paste" "F.Mask") (roundrect_rratio 0.175439)
+    (pad "2" smd roundrect (at 1.4875 0 90) (size 1.425 1.75) (layers "F.Cu" "F.Paste" "F.Mask") (roundrect_rratio 0.1754392982)
       (net 91 "Net-(D118-Pad2)") (pinfunction "A") (pintype "passive"))
   )
