File: dilemma_assembled/dilemma.kicad_sch (KiCad schematic)
At the start: 106 parts, among them J1 USB_C_Receptacle_USB2.0, J102 Serial, J103 Serial, J105 Conn_01x04_Female, J107 Conn_01x08_Female, J108 Conn_01x01_Female, J109 Conn_01x01_Female, J113 Cirque, J5 Conn_01x02, SW1 SW_Push, SW101 SW_Push, SW102 SW_Push, SW103 SW_Push, SW104 SW_Push, SW105 SW_Push, SW106 SW_Push, SW107 SW_Push, SW108 SW_Push, SW109 SW_Push, SW110 SW_SPST, SW111 SW_SPST, SW112 SW_Push, SW113 SW_Push, SW114 SW_Push, SW115 SW_Push, SW116 SW_Push, SW117 SW_Push, SW118 SW_Push, SW119 SW_Push, SW2 SW_Push, U1 RP2040, U2 GD25Q80CEIGR, U3 XC6210B332MR-G, Y1 Crystal_GND24

Commit message: add 6th column
Parts:
- added D? (x3): D, local-libraries:D_1206_handsolder_reversible, symbol Device:D
- added SW? (x3): SW_Push, local-libraries:SW_MX_choc, symbol Switch:SW_Push
Connections:
- net row2_l: now also SW?.1
- net row3_l: now also SW?.1
- net row4_l: now also SW?.1
- net D12 renamed col6_l
- net col6_l: now also D?.1 (K), D?.1 (K), D?.1 (K)
- new net: D?.2 (A), SW?.2 (x3)
- no-connect marks 20 -> 19
Other:
- moved on the sheet: D101, D102, D103, D104, D105, D106, D107, D108, D109, D110, D111, D112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
