File: dilemma_assembled/dilemma.kicad_sch (KiCad schematic)
At the start: 112 parts, among them J1 USB_C_Receptacle_USB2.0, J102 Serial, J103 Serial, J105 Conn_01x04_Female, J107 Conn_01x08_Female, J108 Conn_01x01_Female, J109 Conn_01x01_Female, J113 Cirque, J5 Conn_01x02, SW1 SW_Push, SW101 SW_Push, SW102 SW_Push, SW103 SW_Push, SW104 SW_Push, SW105 SW_Push, SW106 SW_Push, SW107 SW_Push, SW108 SW_Push, SW109 SW_Push, SW110 SW_SPST, SW111 SW_SPST, SW112 SW_Push, SW113 SW_Push, SW114 SW_Push, SW115 SW_Push, SW116 SW_Push, SW117 SW_Push, SW118 SW_Push, SW119 SW_Push, SW2 SW_Push, U1 RP2040, U2 GD25Q80CEIGR, U3 XC6210B332MR-G, Y1 Crystal_GND24

Commit message: annotate schematic
Parts:
- gave numbers to parts that had none: 6
Changed lines of the file:
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@@
   (symbol (lib_id "Switch:SW_Push") (at 124.46 255.27 0) (unit 1)
     (in_bom yes) (on_board yes)
-    (property "Reference" "SW?" (id 0) (at 124.46 247.65 0))
+    (property "Reference" "SW122" (id 0) (at 124.46 247.65 0))
     (property "Value" "SW_Push" (id 1) (at 124.46 250.19 0))
     (property "Footprint" "local-libraries:SW_MX_choc" (id 2) (at 124.46 250.19 0)
@@
   (symbol (lib_id "Device:D") (at 134.62 255.27 180) (unit 1)
     (in_bom yes) (on_board yes)
-    (property "Reference" "D?" (id 0) (at 132.715 252.73 90)
+    (property "Reference" "D120" (id 0) (at 132.715 252.73 90)
       (effects (font (size 1.27 1.27)) (justify right))
     )
@@
   (symbol (lib_id "Device:D") (at 134.62 234.95 180) (unit 1)
     (in_bom yes) (on_board yes)
-    (property "Reference" "D?" (id 0) (at 132.715 232.41 90)
+    (property "Reference" "D118" (id 0) (at 132.715 232.41 90)
       (effects (font (size 1.27 1.27)) (justify right))
     )
@@
   (symbol (lib_id "Switch:SW_Push") (at 124.46 234.95 0) (unit 1)
     (in_bom yes) (on_board yes)
-    (property "Reference" "SW?" (id 0) (at 124.46 227.33 0))
+    (property "Reference" "SW120" (id 0) (at 124.46 227.33 0))
     (property "Value" "SW_Push" (id 1) (at 124.46 229.87 0))
     (property "Footprint" "local-libraries:SW_MX_choc" (id 2) (at 124.46 229.87 0)
@@
   (symbol (lib_id "Switch:SW_Push") (at 124.46 245.11 0) (unit 1)
     (in_bom yes) (on_board yes)
-    (property "Reference" "SW?" (id 0) (at 124.46 237.49 0))
+    (property "Reference" "SW121" (id 0) (at 124.46 237.49 0))
     (property "Value" "SW_Push" (id 1) (at 124.46 240.03 0))
     (property "Footprint" "local-libraries:SW_MX_choc" (id 2) (at 124.46 240.03 0)
@@
   (symbol (lib_id "Device:D") (at 134.62 245.11 180) (unit 1)
     (in_bom yes) (on_board yes)
-    (property "Reference" "D?" (id 0) (at 132.715 242.57 90)
+    (property "Reference" "D119" (id 0) (at 132.715 242.57 90)
       (effects (font (size 1.27 1.27)) (justify right))
     )
@@
       (reference "D117") (unit 1) (value "D") (footprint "local-libraries:D_1206_handsolder_reversible")
     )
-    (path "/3f89b463-d3d1-4e4b-986f-c05d51f58a38"
-      (reference "D?") (unit 1) (value "D") (footprint "local-libraries:D_1206_handsolder_reversible")
-    )
     (path "/727f97ca-0e92-4646-88f0-91e2a4c7207c"
-      (reference "D?") (unit 1) (value "D") (footprint "local-libraries:D_1206_handsolder_reversible")
+      (reference "D118") (unit 1) (value "D") (footprint "local-libraries:D_1206_handsolder_reversible")
     )
     (path "/e479d062-53cb-4cef-b140-4bdae47046cc"
-      (reference "D?") (unit 1) (value "D") (footprint "local-libraries:D_1206_handsolder_reversible")
+      (reference "D119") (unit 1) (value "D") (footprint "local-libraries:D_1206_handsolder_reversible")
+    )
+    (path "/3f89b463-d3d1-4e4b-986f-c05d51f58a38"
+      (reference "D120") (unit 1) (value "D") (footprint "local-libraries:D_1206_handsolder_reversible")
     )
     (path "/ce9365fe-085a-4731-86d8-fc3e6b16f716"
@@
       (reference "SW119") (unit 1) (value "SW_Push") (footprint "local-libraries:SW_MX_choc")
     )
-    (path "/0397a46e-b231-4278-b35c-fbeb4dfde2fc"
-      (reference "SW?") (unit 1) (value "SW_Push") (footprint "local-libraries:SW_MX_choc")
-    )
     (path "/cfd6d7d9-e276-49ef-829b-32515e258b69"
-      (reference "SW?") (unit 1) (value "SW_Push") (footprint "local-libraries:SW_MX_choc")
+      (reference "SW120") (unit 1) (value "SW_Push") (footprint "local-libraries:SW_MX_choc")
     )
     (path "/e16d14b5-09e0-413d-bf9e-c02fd14a7dee"
-      (reference "SW?") (unit 1) (value "SW_Push") (footprint "local-libraries:SW_MX_choc")
+      (reference "SW121") (unit 1) (value "SW_Push") (footprint "local-libraries:SW_MX_choc")
+    )
+    (path "/0397a46e-b231-4278-b35c-fbeb4dfde2fc"
+      (reference "SW122") (unit 1) (value "SW_Push") (footprint "local-libraries:SW_MX_choc")
     )
     (path "/073e7a20-6222-4c9d-9f89-871bf718b9fb"
